File: projects/Adaptor Boards/pycubed_non_ext.brd (EAGLE design)
At the start: 90.1 x 115.9 mm, 13 parts, among them J1 M22-6013005

Commit message: Updated PCB Designs
Parts:
- removed H5, H6, H7, H8: MOUNT-PAD-ROUND3.2, holes:3,2-PAD
- moved H3 20.0 mm to (8.89, 90.8)
- moved H4 20.0 mm to (82.5, 90.8)
- moved J1 20.0 mm to (16.5, 84.8)
Routing:
- net PA31: track 76.8 -> 56.8 mm
- net GND1: track 56.6 -> 36.6 mm
- net PA02: track 76.8 -> 56.8 mm
- net GND3: track 83.3 -> 63.3 mm
- net PB22: track 51.0 -> 31.0 mm
- net RESET: track 79.6 -> 59.6 mm
- net PB23: track 50.8 -> 30.8 mm
- net PA20: track 51.2 -> 31.2 mm
- net PA19: track 52.1 -> 32.1 mm
- net PA18: track 52.3 -> 32.3 mm
- net PA17: track 52.5 -> 32.5 mm
- net PA14: track 50.5 -> 30.5 mm
- net PA12: track 50.3 -> 30.3 mm
- net PA05: track 78.9 -> 58.9 mm
- net GND2: track 89.6 -> 69.6 mm
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Other:
- board size 90.1 x 115.9 mm -> 90 x 97 mm
