File: projects/Adaptor Boards/pycubed.brd (EAGLE design)
At the start: 90.1 x 115.9 mm, 13 parts, among them J1 M22-6013005

Commit message: Updated PCB desgins to fix wiring mismatches
Parts:
- moved BOTTOMRIGHT 0.06 mm to (54.7, 33.7), turned to 180 degrees
Connections:
- new net GNDJTAG: BOTTOMLEFT.1, J1.P$115
- net GND2: no longer BOTTOMLEFT.1
- net GND8: no longer J1.P$46
Routing:
- net GNDJTAG: track 0.00 -> 114.6 mm
- net GND2: track 89.6 -> 0.00 mm
- net 3V34: track 81.0 -> 108.8 mm
- net PA05: track 78.9 -> 97.8 mm
- net PA04: track 77.8 -> 92.1 mm
- net GND3: track 83.3 -> 89.7 mm
- net PA02: track 76.8 -> 81.0 mm
Other:
- board text added: "C:/Users/Conor Begley/Documents/EAGLE/projects/FlatSat/glasgow-caledonian-logoW.bmp"
- board text added: "Demo Payload Board Conor Begley MEng 2020-21"
