File: projects/PC104 Cards/Old/com_board.brd (EAGLE design)
At the start: 90 x 97 mm, 7 parts, among them J2 M22-6013005, U2 ESP32-DEVKITC-32D

Commit message: Updated PCB Designs
Parts:
- added SV1: (no value), con-lsta:FE08
- moved SV2 99.2 mm to (10.5, -8.80), turned to 0 degrees
Connections:
- net D18: now also SV1.3
- net D19: now also SV1.2
- net D2: now also SV1.1
- net D21: now also SV1.5
- net D22: now also SV1.6
- net D23: now also SV1.8
- net D4: now also SV1.4
- net GND1: now also SV1.7
Routing:
- net GND2: track 67.2 -> 0.00 mm
- net D2: track 74.3 -> 66.9 mm
- net D21: track 69.4 -> 67.3 mm
- net D19: track 152.6 -> 150.5 mm
- net D4: track 112.0 -> 109.9 mm
- net D22: track 65.1 -> 63.0 mm
- net D18: track 135.9 -> 133.8 mm
- net D23: track 47.1 -> 48.2 mm
- net GND4: track 74.9 -> 74.1 mm
