File: projects/PC104 Cards/Old/com_board.sch (EAGLE design)
At the start: 13 parts, among them J1 M22-6013005

Commit message: Updated PCB Designs
Parts:
- removed BOTTOMLEFT, BOTTOMRIGHT, TOPRIGHT: (no value), con-lstb:MA05-1
- removed H5, H6, H7, H8: MOUNT-PAD-ROUND3.2, holes:MOUNT-PAD-ROUND3.2
- removed J1: M22-6013005, M22-6013005:M22-6013005
- removed TOPLEFT: (no value), con-lstb:MA09-1
- added J2: M22-6013005, M22-6013005:M22-6013005
- added SV1: (no value), con-lsta:FE08-1
- added SV2: (no value), con-lsta:FE12-1
- added U2: ESP32-DEVKITC-32D, ESP32-DEVKITC-32D:ESP32-DEVKITC-32D
Connections:
- removed net 3V33: BOTTOMLEFT.5, J1.A9
- removed net 3V34: BOTTOMRIGHT.1, J1.A18
- removed net PA02: BOTTOMRIGHT.5, J1.A21
- removed net PA04: BOTTOMRIGHT.4, J1.A20
- removed net PA05: BOTTOMRIGHT.3, J1.A19
- removed net PA12: J1.A3, TOPLEFT.4
- removed net PA13: J1.A2, TOPLEFT.3
- removed net PA14: J1.A4, TOPLEFT.5
- removed net PA17: J1.A17, TOPRIGHT.5
- removed net PA18: J1.A16, TOPRIGHT.4
- removed net PA19: J1.A15, TOPRIGHT.3
- removed net PA20: J1.A7, TOPLEFT.8
- removed net PA22: J1.A8, TOPLEFT.9
- removed net PA30: BOTTOMLEFT.4, J1.A10
- removed net PA31: BOTTOMLEFT.3, J1.A11
- removed net PB16: J1.A14, TOPRIGHT.2
- removed net PB17: J1.A13, TOPRIGHT.1
- removed net PB22: J1.A6, TOPLEFT.7
- removed net PB23: J1.A5, TOPLEFT.6
- removed net RESET: BOTTOMLEFT.2, J1.A12
- new net ADC: J2.A21
- new net ADC2: U2.IO4
- new net D18: SV1.3, SV2.4, U2.IO13
- new net D19: SV1.2, SV2.3, U2.IO14
- new net D2: SV1.1, SV2.2, U2.IO5
- new net D21: SV1.5, SV2.6, U2.IO15
- new net D22: SV1.6, SV2.7, U2.IO2
- new net D23: SV1.8, SV2.12, U2.IO0
- new net D4: SV1.4, SV2.5, U2.IO27
- new net D5: U2.IO12
- new net DAC1: J2.A19, U2.IO25
- new net DAC2: J2.A20, U2.IO26
- new net EN: U2.EN
- new net GPIO: J2.A5
- new net GPIO1: J2.A6, U2.SENSOR_VP
- new net GPIO2: J2.A7, U2.SENSOR_VN
- new net GPIO3: J2.A8, U2.IO34
- new net GPIO4: J2.A15, U2.IO35
- new net GPIO5: J2.A16, U2.IO32
- new net GPIO6: J2.A17, U2.IO33
- new net MISO: J2.A4, U2.IO19
- new net RX: J2.A3, U2.IO23, U2.RXD0
- new net SCL: J2.A14, U2.IO17, U2.IO22
- new net SDA: J2.A13, U2.IO16, U2.IO21
- new net TX: J2.A2, U2.IO18, U2.TXD0
- net 12V: now also J2.C12; no longer J1.C12
- net 12V1: now also J2.D12; no longer J1.D12
- net 3V3: now also J2.C14; no longer J1.D14
- net 3V31: now also J2.D14; no longer J1.C14
- net 3V32: now also U2.3V3; no longer J1.A1, TOPLEFT.1
- net 5V: now also J2.C13, U2.EXT_5V; no longer J1.D13
- net 5V1: now also J2.D13; no longer J1.C13
- net GND1: now also SV1.7, SV2.11; no longer J1.C5, TOPLEFT.2
- net GND10: now also J2.D24; no longer J1.D24
- net GND2: now also J2.D7, SV2.10; no longer BOTTOMLEFT.1, J1.D7
- net GND3: now also J2.C9, U2.GND1; no longer BOTTOMRIGHT.2, J1.C9
- net GND4: now also J2.C11, U2.GND2; no longer J1.C11
- net GND5: now also J2.D11, U2.GND3; no longer J1.D11
- net GND6: now also J2.C15; no longer J1.C15
- net GND7: now also J2.D15; no longer J1.D15
- net GND8: now also J2.D16; no longer J1.C16, J1.D16
- net GND9: now also J2.C24; no longer J1.C24
