File: projects/FlatSat/FlatSat_Final.brd (EAGLE design)
At the start: 290 x 267 mm, 46 parts, among them J1 M22-6013005, J2 M22-6013005, J3 M22-6013005, J4 M22-6013005, J5 M22-6013005, J6 M22-6013005

Commit message: Updated PCB desgins to fix wiring mismatches
Routing:
- net VBAT: track 642.4 -> 635.4 mm
- net +3.3V: track 666.3 -> 659.9 mm
- net +5V: track 674.2 -> 668.4 mm
- net +12V: track 682.6 -> 677.4 mm
- net H2-19: track 851.7 -> 850.2 mm
- net H1-16: track 828.9 -> 827.9 mm
- net UN13: track 1250.3 -> 1249.4 mm
- net UN11: track 1222.7 -> 1221.8 mm
- net UN02: track 1315.9 -> 1314.9 mm
- net H2-41: track 1065.4 -> 1064.5 mm
- net H1-40: track 1159.8 -> 1158.9 mm
- net H1-38: track 1132.2 -> 1131.3 mm
- net H1-32: track 1049.6 -> 1048.7 mm
- net H1-26: track 966.8 -> 965.9 mm
- net UN15: track 1277.9 -> 1277.0 mm
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Other:
- board text added: "3V3"
