File: projects/FlatSat/OLD/FlatSat_Final.brd (EAGLE design)
At the start: 290 x 267 mm, 46 parts, among them J1 M22-6013005, J2 M22-6013005, J3 M22-6013005, J4 M22-6013005, J5 M22-6013005, J6 M22-6013005

Commit message: Updated PCB desgins to fix wiring mismatches
Routing:
- net H2-19: track 851.7 -> 850.2 mm
- net H1-16: track 828.9 -> 827.9 mm
- net UN13: track 1250.3 -> 1249.4 mm
- net UN11: track 1222.7 -> 1221.8 mm
- net UN02: track 1315.9 -> 1314.9 mm
- net H2-41: track 1065.4 -> 1064.5 mm
- net H1-40: track 1159.8 -> 1158.9 mm
- net H1-38: track 1132.2 -> 1131.3 mm
- net H1-32: track 1049.6 -> 1048.7 mm
- net H1-26: track 966.8 -> 965.9 mm
- net UN15: track 1277.9 -> 1277.0 mm
- net UN06: track 1356.3 -> 1355.4 mm
- net H2-51: track 1167.5 -> 1166.5 mm
- net H2-35: track 982.7 -> 981.8 mm
- net H2-31: track 927.6 -> 926.6 mm
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