File: projects/PC104 Cards/com_board.brd (EAGLE design)
At the start: 90 x 97 mm, 7 parts, among them J2 M22-6013005, U2 ESP32-DEVKITC-32D

Commit message: Updated PCB desgins to fix wiring mismatches
Parts:
- removed SV2: (no value), con-lsta:FE12
- added SV1: (no value), con-lsta:FE09
Connections:
- removed net ADC2: U2.32
- removed net D18: SV2.4, U2.15
- removed net D19: SV2.3, U2.12
- removed net D21: SV2.6, U2.35
- removed net D22: SV2.7, U2.34
- removed net D23: SV2.12, U2.33
- removed net D4: SV2.5, U2.11
- removed net D5: U2.13
- removed net EN: U2.2
- removed net GND1: SV2.11
- new net CS: SV1.3, U2.35
- new net DC: SV1.5, U2.33
- new net DON'TCONNECT: U2.20
- new net GND_ESP: SV1.2, U2.14
- new net LCD_CLK: SV1.7, U2.12
- new net LCD_MISO: SV1.9, U2.15
- new net LCD_MOSI: SV1.6, U2.13
- new net LED: SV1.8, U2.34
- new net RESET: SV1.4, U2.11
- net 3V32: now also SV1.1
- net ADC: now also U2.32
- net D2: no longer SV2.2
- net GND2: no longer SV2.10
- net GND3: now also U2.26; no longer U2.14
- net GND4: no longer U2.26
- net GND5: no longer U2.20
- net GPIO: now also U2.2
- net SCL: now also J2.P$103; no longer J2.P$104
- net SDA: now also J2.P$104; no longer J2.P$103
Routing:
- net 3V32: track 0.00 -> 188.1 mm
- net D19: track 152.6 -> 0.00 mm
- net D18: track 135.9 -> 0.00 mm
- net GND_ESP: track 0.00 -> 115.7 mm
- net D4: track 112.0 -> 0.00 mm
- net RESET: track 0.00 -> 106.4 mm
- net LCD_MOSI: track 0.00 -> 87.4 mm
- net LCD_MISO: track 0.00 -> 85.9 mm
- net LCD_CLK: track 0.00 -> 82.6 mm
- net GND4: track 74.9 -> 0.00 mm
- net D2: track 74.3 -> 0.00 mm
- net CS: track 0.00 -> 73.9 mm
- net D21: track 69.4 -> 0.00 mm
- net GND2: track 67.2 -> 0.00 mm
- net DC: track 0.00 -> 65.9 mm
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Other:
- board text added: "C:/Users/Conor Begley/Documents/EAGLE/projects/FlatSat/glasgow-caledonian-logoW.bmp"
- board text added: "Demo Communication Board Conor Begley MEng 2020-21"
