File: projects/PC104 Cards/demo_board.sch (EAGLE design)
At the start: 17 parts, among them J2 M22-6013005, U2 ESP32-DEVKITC-32D

Commit message: Updated PCB desgins to fix wiring mismatches
Connections:
- removed net ADC2: U2.IO4
- removed net EN: U2.EN
- removed net N$2: R4.1, R5.1
- new net DONTCONNECT: U2.GND3
- net 3V3: now also R4.2
- net ADC: now also U2.IO4
- net GND5: no longer U2.GND3
- net GPIO: now also U2.EN; no longer U2.IO5
- net SCL: now also J2.A13; no longer J2.A14
- net SDA: now also J2.A14; no longer J2.A13
- net THERM: now also R4.1, R5.1; no longer R4.2
